Commit message: fix:gen3 urdf

File: content/assets/urdf/kinova_description/gen3.urdf (robot description, URDF)
Before this commit: robot gen3, 9 links, 8 joints
Joints:
- joint joint_1: type continuous -> revolute
- joint joint_3: type continuous -> revolute
- joint joint_5: type continuous -> revolute
- joint joint_7: type continuous -> revolute
